Commit message: Added prefixing for dual arm support for m1013

File: dsr_description2/config/macro.materials.xacro (robot description, xacro)
@@ -1,27 +1,29 @@
 <?xml version="1.0"?>
 <robot name="dsr_materials" xmlns:xacro="http://www.ros.org/wiki/xacro">
-	<xacro:macro name="dsr_materials">
-		<material name="black">
+	<xacro:macro name="dsr_materials" params="
+		tf_prefix:=''
+		">
+		<material name="${tf_prefix}black">
 			<color rgba="0.0 0.0 0.0 1.0" />
 		</material>
-		<material name="white">
+		<material name="${tf_prefix}white">
 			<color rgba="1.0 1.0 1.0 1.0" />
 		</material>
-		<material name="orange">
+		<material name="${tf_prefix}orange">
 			<color rgba="1.0 0.4 0.0 1.0" />
 		</material>
-		<material name="dr_gray">
+		<material name="${tf_prefix}dr_gray">
 			<color rgba="0.490 0.490 0.486 1.0" />
 		</material>
-		<material name="dr_white">
+		<material name="${tf_prefix}dr_white">
 			<color rgba="0.941 0.941 0.941 1.0" />
 		</material>
-		<material name="dr_blue">
+		<material name="${tf_prefix}dr_blue">
 			<color rgba="0 0 0.15 1" />
 		</material>
-		<material name="grey">
+		<material name="${tf_prefix}grey">
 			<color rgba="0.5 0.5 0.5 1.0" />
 		</material>
-		<material name="Boxer_DarkGrey">
+		<material name="${tf_prefix}Boxer_DarkGrey">
 			<color rgba="0.3 0.3 0.3 1.0" />
 		</material>

File: dsr_description2/ros2_control/m1013.ros2_control.xacro (robot description, xacro)
@@ -3,26 +3,35 @@
   <!-- Doosan M1013 ros2_control (arm-only) -->
   <xacro:macro name="m1013_ros2_control" params="
-  name
-  host:=0.0.0.0
-  rt_host:=0.0.0.0
-  port:=12345
-  mode:=real
-  model:=m1013
-  update_rate
-  ">
+      name
+      tf_prefix:=''
+      use_mock_hw:=false
+      rate:=100
+      standby:=true
+      command:=none
+      host:=0.0.0.0
+      rt_host:=0.0.0.0
+      port:=12345
+      mode:=real
+      model:=m1013
+      update_rate">
     <xacro:property name="double_pi" value="${2.0 * pi}"/>
     <xacro:property name="neg_double_pi" value="${-2.0 * pi}"/>
     <ros2_control name="${name}" type="system">
       <hardware>
-        <plugin>dsr_hardware2/DRHWInterface</plugin>
-        <param name="host">${host}</param>
-        <param name="rt_host">${rt_host}</param>
-        <param name="port">${port}</param>
-        <param name="mode">${mode}</param>
-        <param name="model">${model}</param>
-        <param name="update_rate">${update_rate}</param>
+        <xacro:if value="${use_mock_hw}">
+          <plugin>mock_components/GenericSystem</plugin>
+        </xacro:if>
+        <xacro:unless value="${use_mock_hw}">
+          <plugin>dsr_hardware2/DRHWInterface</plugin>
+          <param name="host">${host}</param>
+          <param name="rt_host">${rt_host}</param>
+          <param name="port">${port}</param>
+          <param name="mode">${mode}</param>
+          <param name="model">${model}</param>
+          <param name="update_rate">${update_rate}</param>
+        </xacro:unless>
       </hardware>
       <!-- Arm joints only -->
-      <joint name="joint_1">
+      <joint name="${tf_prefix}joint_1">
         <command_interface name="position">
           <param name="min">${neg_double_pi}</param>
@@ -36,5 +45,5 @@
         <state_interface name="velocity"/>
       </joint>
-      <joint name="joint_2">
+      <joint name="${tf_prefix}joint_2">
         <command_interface name="position">
           <param name="min">${neg_double_pi}</param>
@@ -48,5 +57,5 @@
         <state_interface name="velocity"/>
       </joint>
-      <joint name="joint_3">
+      <joint name="${tf_prefix}joint_3">
         <command_interface name="position">
           <param name="min">${neg_double_pi}</param>
@@ -60,5 +69,5 @@
         <state_interface name="velocity"/>
       </joint>
-      <joint name="joint_4">
+      <joint name="${tf_prefix}joint_4">
         <command_interface name="position">
           <param name="min">${neg_double_pi}</param>
@@ -72,5 +81,5 @@
         <state_interface name="velocity"/>
       </joint>
-      <joint name="joint_5">
+      <joint name="${tf_prefix}joint_5">
         <command_interface name="position">
           <param name="min">${neg_double_pi}</param>
@@ -84,5 +93,5 @@
         <state_interface name="velocity"/>
       </joint>
-      <joint name="joint_6">
+      <joint name="${tf_prefix}joint_6">
         <command_interface name="position">
           <param name="min">${neg_double_pi}</param>

File: dsr_description2/xacro/macro.m1013.blue.xacro (robot description, xacro)
@@ -4,7 +4,12 @@
 	<xacro:include filename="$(find dsr_description2)/config/macro.transmission.xacro" />
 	<xacro:include filename="$(find dsr_description2)/config/macro.materials.xacro" />
-	<xacro:macro name="m1013" params="namespace simple:=false">
-		<xacro:dsr_materials />
-		<link name="base_link">
+	<xacro:macro name="m1013" params="
+		namespace
+		simple:=false
+		name:='m1013'
+		tf_prefix:=''
+		">
+		<xacro:dsr_materials tf_prefix="${tf_prefix}"/>
+		<link name="${tf_prefix}base_link">
 			<inertial>
 				<mass value="4.12"/>
@@ -28,7 +33,7 @@
 		</link>
 		<!-- joint 1 -->
-		<joint name="joint_1" type="revolute">
-			<parent link="base_link" />
-			<child link="link_1" />
+		<joint name="${tf_prefix}joint_1" type="revolute">
+			<parent link="${tf_prefix}base_link" />
+			<child link="${tf_prefix}link_1" />
 			<origin rpy="0 0 0" xyz="0 0 0.1525" />
 			<axis xyz="0 0 1" />
@@ -36,5 +41,5 @@
 			<dynamics friction="0" />
 		</joint>
-		<link name="link_1">
+		<link name="${tf_prefix}link_1">
 			<inertial>
 				<mass value="7.8"/>
@@ -58,7 +63,7 @@
 		</link>
 		<!-- joint2 -->
-		<joint name="joint_2" type="revolute">
-			<parent link="link_1" />
-			<child link="link_2" />
+		<joint name="${tf_prefix}joint_2" type="revolute">
+			<parent link="${tf_prefix}link_1" />
+			<child link="${tf_prefix}link_2" />
 			<origin rpy="0 -1.571 -1.571" xyz="0 0.0345 0" />
 			<axis xyz="0 0 1" />
@@ -66,5 +71,5 @@
 			<dynamics friction="0" />
 		</joint>
-		<link name="link_2">
+		<link name="${tf_prefix}link_2">
 			<inertial>
 				<mass value="10.83"/>
@@ -112,7 +117,7 @@
 		</link>
 		<!-- joint3 -->
-		<joint name="joint_3" type="revolute">
-			<parent link="link_2" />
-			<child link="link_3" />
+		<joint name="${tf_prefix}joint_3" type="revolute">
+			<parent link="${tf_prefix}link_2" />
+			<child link="${tf_prefix}link_3" />
 			<origin rpy="0 0 1.571" xyz="0.62 0 0" />
 			<axis xyz="0 0 1" />
@@ -120,5 +125,5 @@
 			<dynamics friction="0" />
 		</joint>
-		<link name="link_3">
+		<link name="${tf_prefix}link_3">
 			<inertial>
 				<mass value="3.68"/>
@@ -142,7 +147,7 @@
 		</link>
 		<!-- joint4 -->
-		<joint name="joint_4" type="revolute">
-			<parent link="link_3" />
-			<child link="link_4" />
+		<joint name="${tf_prefix}joint_4" type="revolute">
+			<parent link="${tf_prefix}link_3" />
+			<child link="${tf_prefix}link_4" />
 			<origin rpy="1.571 0 0" xyz="0 -0.559 0" />
 			<axis xyz="0 0 1" />
@@ -150,5 +155,5 @@
 			<dynamics friction="0" />
 		</joint>
-		<link name="link_4">
+		<link name="${tf_prefix}link_4">
 			<inertial>
 				<mass value="3.82"/>
@@ -183,7 +188,7 @@
 		</link>
 		<!-- joint5 -->
-		<joint name="joint_5" type="revolute">
-			<parent link="link_4" />
-			<child link="link_5" />
+		<joint name="${tf_prefix}joint_5" type="revolute">
+			<parent link="${tf_prefix}link_4" />
+			<child link="${tf_prefix}link_5" />
 			<origin rpy="-1.571 0 0" xyz="0 0 0" />
 			<axis xyz="0 0 1" />
@@ -191,5 +196,5 @@
 			<dynamics friction="0" />
 		</joint>
-		<link name="link_5">
+		<link name="${tf_prefix}link_5">
 			<inertial>
 				<mass value="2.82"/>
@@ -213,7 +218,7 @@
 		</link>
 		<!-- joint6 -->
-		<joint name="joint_6" type="revolute">
-			<parent link="link_5" />
-			<child link="link_6" />
+		<joint name="${tf_prefix}joint_6" type="revolute">
+			<parent link="${tf_prefix}link_5" />
+			<child link="${tf_prefix}link_6" />
 			<origin rpy="1.571 0 0" xyz="0 -0.121 0" />
 			<axis xyz="0 0 1" />
@@ -221,5 +226,5 @@
 			<dynamics friction="0" />
 		</joint>
-		<link name="link_6">
+		<link name="${tf_prefix}link_6">
 			<inertial>
 				<mass value="1.16"/>

File: dsr_description2/xacro/macro.m1013.white.xacro (robot description, xacro)
@@ -4,7 +4,12 @@
 	<xacro:include filename="$(find dsr_description2)/config/macro.transmission.xacro" />
 	<xacro:include filename="$(find dsr_description2)/config/macro.materials.xacro" />
-	<xacro:macro name="m1013" params="namespace simple:=false">
-		<xacro:dsr_materials />
-		<link name="base_link">
+	<xacro:macro name="m1013" params="
+		namespace
+		simple:=false
+		name:='m1013'
+		tf_prefix:=''
+		">
+		<xacro:dsr_materials tf_prefix="${tf_prefix}"/>
+		<link name="${tf_prefix}base_link">
 			<inertial>
 				<mass value="4.12"/>
@@ -28,7 +33,7 @@
 		</link>
 		<!-- joint 1 -->
-		<joint name="joint_1" type="revolute">
-			<parent link="base_link" />
-			<child link="link_1" />
+		<joint name="${tf_prefix}joint_1" type="revolute">
+			<parent link="${tf_prefix}base_link" />
+			<child link="${tf_prefix}link_1" />
 			<origin rpy="0 0 0" xyz="0 0 0.1525" />
 			<axis xyz="0 0 1" />
@@ -36,5 +41,5 @@
 			<dynamics friction="0" />
 		</joint>
-		<link name="link_1">
+		<link name="${tf_prefix}link_1">
 			<inertial>
 				<mass value="7.8"/>
@@ -58,7 +63,7 @@
 		</link>
 		<!-- joint2 -->
-		<joint name="joint_2" type="revolute">
-			<parent link="link_1" />
-			<child link="link_2" />
+		<joint name="${tf_prefix}joint_2" type="revolute">
+			<parent link="${tf_prefix}link_1" />
+			<child link="${tf_prefix}link_2" />
 			<origin rpy="0 -1.571 -1.571" xyz="0 0.0345 0" />
 			<axis xyz="0 0 1" />
@@ -66,5 +71,5 @@
 			<dynamics friction="0" />
 		</joint>
-		<link name="link_2">
+		<link name="${tf_prefix}link_2">
 			<inertial>
 				<mass value="10.83"/>
@@ -112,7 +117,7 @@
 		</link>
 		<!-- joint3 -->
-		<joint name="joint_3" type="revolute">
-			<parent link="link_2" />
-			<child link="link_3" />
+		<joint name="${tf_prefix}joint_3" type="revolute">
+			<parent link="${tf_prefix}link_2" />
+			<child link="${tf_prefix}link_3" />
 			<origin rpy="0 0 1.571" xyz="0.62 0 0" />
 			<axis xyz="0 0 1" />
@@ -120,5 +125,5 @@
 			<dynamics friction="0" />
 		</joint>
-		<link name="link_3">
+		<link name="${tf_prefix}link_3">
 			<inertial>
 				<mass value="3.68"/>
@@ -142,7 +147,7 @@
 		</link>
 		<!-- joint4 -->
-		<joint name="joint_4" type="revolute">
-			<parent link="link_3" />
-			<child link="link_4" />
+		<joint name="${tf_prefix}joint_4" type="revolute">
+			<parent link="${tf_prefix}link_3" />
+			<child link="${tf_prefix}link_4" />
 			<origin rpy="1.571 0 0" xyz="0 -0.559 0" />
 			<axis xyz="0 0 1" />
@@ -150,5 +155,5 @@
 			<dynamics friction="0" />
 		</joint>
-		<link name="link_4">
+		<link name="${tf_prefix}link_4">
 			<inertial>
 				<mass value="3.82"/>
@@ -183,7 +188,7 @@
 		</link>
 		<!-- joint5 -->
-		<joint name="joint_5" type="revolute">
-			<parent link="link_4" />
-			<child link="link_5" />
+		<joint name="${tf_prefix}joint_5" type="revolute">
+			<parent link="${tf_prefix}link_4" />
+			<child link="${tf_prefix}link_5" />
 			<origin rpy="-1.571 0 0" xyz="0 0 0" />
 			<axis xyz="0 0 1" />
@@ -191,5 +196,5 @@
 			<dynamics friction="0" />
 		</joint>
-		<link name="link_5">
+		<link name="${tf_prefix}link_5">
 			<inertial>
 				<mass value="2.82"/>
@@ -213,7 +218,7 @@
 		</link>
 		<!-- joint6 -->
-		<joint name="joint_6" type="revolute">
-			<parent link="link_5" />
-			<child link="link_6" />
+		<joint name="${tf_prefix}joint_6" type="revolute">
+			<parent link="${tf_prefix}link_5" />
+			<child link="${tf_prefix}link_6" />
 			<origin rpy="1.571 0 0" xyz="0 -0.121 0" />
 			<axis xyz="0 0 1" />
@@ -221,5 +226,5 @@
 			<dynamics friction="0" />
 		</joint>
-		<link name="link_6">
+		<link name="${tf_prefix}link_6">
 			<inertial>
 				<mass value="1.16"/>
